Commit message: Debugged the cylinders issue at the effector

File: robot_description/urdf/Jaco_def.urdf (robot description, URDF)
Before this commit: robot Jaco, 7 links, 6 joints
Joints:
- joint joint_1: origin xyz=0 0 0 rpy=0 0 0 -> xyz=0 0 0.1455 rpy=0 0 0
- joint joint_6: origin xyz=0 0 0.0741 rpy=0 0 0 -> xyz=0 0 0.0741 rpy=0 1.0472 0

Commit message: Added inertia to links and corrected geometry

File: robot_description/urdf/Jaco_def.urdf (robot description, URDF)
Before this commit: robot Jaco, 7 links, 6 joints
Links:
- link base_link: mass None -> 0.601719; geometry visual cylinder length=0.1579 radius=0.03
- link effector: mass None -> 0.604973
- link link_2: mass None -> 0.7872084; geometry visual cylinder length=0.1176 radius=0.03
- link link_3: mass None -> 1.205432
- link link_4: mass None -> 0.89128
- link link_5: mass None -> 0.471842
- link link_6: mass None -> 0.471842
Joints:
- joint joint_1: origin xyz=0 0 0.1455 rpy=0 0 0 -> xyz=0 0 0.1579 rpy=0 0 0
- joint joint_2: origin xyz=0 0 0.13 rpy=0 0 0 -> xyz=0 0 0.1176 rpy=0 0 0

Commit message: Added a plugin for gazebo

File: robot_description/urdf/Jaco_def.urdf (robot description, URDF)
Before this commit: robot Jaco, 7 links, 6 joints
Links:
- added link world
Joints:
- added joint fixed: type fixed, parent world, child base_link

Commit message: added meshes for the wrist and updated the urdf

File: robot_description/urdf/Jaco_def.urdf (robot description, URDF)
Before this commit: robot Jaco, 8 links, 7 joints
Links:
- link link_5: geometry visual mesh filename=file://$(find robot_description)/meshes/wrist.STL
- link link_6: geometry visual mesh filename=file://$(find robot_description)/meshes/wrist.STL
Joints:
- joint joint_5: origin xyz=0 0 0.0741 rpy=0 -1.0472 0 -> xyz=-0.038 0 0.0631 rpy=0 -1.0472 0
- joint joint_6: origin xyz=0 0 0.0741 rpy=0 1.0472 0 -> xyz=0.038 0.0 0.0631 rpy=0 1.0472 0

Commit message: old version

File: robot_description/urdf/Jaco_def.urdf (robot description, URDF)
Before this commit: robot Jaco, 8 links, 7 joints
Links:
- removed link world
- link base_link: mass 0.601719 -> None
Joints:
- removed joint fixed

Commit message: Clean up the gazebo launch

File: robot_description/urdf/Jaco_def.urdf (robot description, URDF)
Before this commit: robot Jaco, 7 links, 6 joints
Links:
- link base_link: geometry collision cylinder length=0.10 radius=0.03; visual cylinder length=0.1579 radius=0.03
