Commit message: Debugged the URDF for gazebo

File: robot_description/urdf/jaco_def.urdf (robot description, URDF)
Before this commit: robot Jaco, 7 links, 6 joints
Links:
- link base_link: mass None -> 0.7872084
- link link_5: geometry visual mesh filename=package://robot_description/meshes/wrist.STL
- link link_6: geometry visual mesh filename=package://robot_description/meshes/wrist.STL

Commit message: Adjusted PID coefficients, except joint 2

File: robot_description/urdf/jaco_def.urdf (robot description, URDF)
Before this commit: robot Jaco, 7 links, 6 joints
Links:
- added link world
Joints:
- added joint fixed: type fixed, parent world, child base_link
- joint joint_1: limit lower=0 upper=6.28319 effort=12 velocity=12.2 -> effort=12 velocity=12.2; type revolute -> continuous
- joint joint_2: limit lower=0 upper=6.28319 effort=12 velocity=12.2 -> effort=1200 velocity=12.2; type revolute -> continuous
- joint joint_3: limit lower=0 upper=6.28319 effort=12 velocity=12.2 -> effort=12 velocity=12.2; type revolute -> continuous
- joint joint_4: limit lower=0 upper=6.28319 effort=3.6 velocity=20.3 -> effort=3.6 velocity=20.3; type revolute -> continuous
- joint joint_5: limit lower=0 upper=6.28319 effort=3.6 velocity=20.3 -> effort=3.6 velocity=20.3; type revolute -> continuous
- joint joint_6: limit lower=0 upper=6.28319 effort=3.6 velocity=20.3 -> effort=3.6 velocity=20.3; type revolute -> continuous

Commit message: Adjusted the PID coefficients

File: robot_description/urdf/jaco_def.urdf (robot description, URDF)
Before this commit: robot Jaco, 8 links, 7 joints
Joints:
- joint joint_2: limit effort=1200 velocity=12.2 -> effort=12 velocity=12.2

Commit message: Added the trajectory experimental file

File: robot_description/urdf/jaco_def.urdf (robot description, URDF)
Before this commit: robot Jaco, 8 links, 7 joints
Links:
- removed link base_link
- added link link_1, mass 0.7872084; collision cylinder length=0.10 radius=0.03; visual cylinder length=0.1579 radius=0.03
Joints:
- joint fixed: child base_link -> link_1
- joint joint_1: parent base_link -> link_1
